File: projects/resistive-load/resistive-load.kicad_pcb (KiCad board)
At the start: 2 copper layers, 236 parts, among them J1 MicroFit_V_2, J2 redcude_7461166, J3 redcude_7461166, J4 redcude_7461166, J5 USB4105-GF-A, J6 Conn_01x20, J7 Conn_01x03, J8 Barrel_jack, Q1 RK7002BMT116, Q10 PJP45N06A_T0_00001, Q11 PJP45N06A_T0_00001, Q12 PJP45N06A_T0_00001, Q13 PJP45N06A_T0_00001, Q14 PJP45N06A_T0_00001, Q15 PJP45N06A_T0_00001, Q16 PJP45N06A_T0_00001, Q17 PJP45N06A_T0_00001, Q18 PJP45N06A_T0_00001, Q19 PJP45N06A_T0_00001, Q2 SSM3J334R, Q20 PJP45N06A_T0_00001, Q21 PJP45N06A_T0_00001, Q22 PJP45N06A_T0_00001, Q23 RK7002BMT116, Q24 SSM3J334R, Q25 SSM3K333R, Q26 RK7002BMT116, Q27 SSM3J334R, Q28 SSM3K333R, Q29 RK7002BMT116, Q3 SSM3K333R, Q30 SSM3J334R, Q31 SSM3K333R, Q32 RK7002BMT116, Q33 SSM3J334R, Q34 SSM3K333R, Q35 SSM3K333R, Q36 SSM3K333R, Q37 SSM3K333R, Q38 SSM3K333R, Q39 SSM3K333R, Q4 PJP45N06A_T0_00001, Q40 RK7002BMT116, Q41 SSM3J334R, Q42 SSM3K333R, Q43 RK7002BMT116, Q44 SSM3J334R, Q45 SSM3K333R, Q46 RK7002BMT116, Q47 SSM3J334R, Q48 SSM3K333R, Q49 RK7002BMT116, Q5 PJP45N06A_T0_00001, Q50 SSM3J334R, Q51 SSM3K333R, Q52 RK7002BMT116, Q53 SSM3J334R, Q54 SSM3K333R, Q55 RK7002BMT116, Q56 SSM3J334R, Q57 SSM3K333R, Q58 RK7002BMT116, Q59 SSM3J334R, Q6 PJP45N06A_T0_00001, Q60 SSM3K333R, Q61 RK7002BMT116, Q62 SSM3J334R, Q63 SSM3K333R, Q64 RK7002BMT116, Q65 SSM3J334R, Q66 SSM3K333R, Q7 PJP45N06A_T0_00001, Q8 PJP45N06A_T0_00001, Q9 PJP45N06A_T0_00001, U1 W25Q128JV, U2 MCP6001, U3 RP2040, U4 MCP1702T-3302E_CB, Y1 12MHz

Commit message: Ayo
Ayo
Parts:
- moved J4 469.9 mm to (447.0, 233.0), turned to 180 degrees
- moved J3 428.9 mm to (420.9, 233.0), turned to 180 degrees
- moved J2 383.6 mm to (396.2, 233.0), turned to 0 degrees
- moved J5 359.5 mm to (339.7, -36.8), turned to 180 degrees
- moved J8 356.3 mm to (358.1, -29.1), turned to -90 degrees
- moved J1 352.6 mm to (367.6, -12.1), turned to 180 degrees
- moved J7 329.3 mm to (369.0, -34.3), turned to 90 degrees
- moved D1 311.0 mm to (351.7, -19.0), turned to 90 degrees
- moved R2 297.9 mm to (352.4, -7.98), turned to 90 degrees
- moved U2 261.5 mm to (348.6, -13.3), turned to -90 degrees
- moved R4 255.3 mm to (349.8, -8.26), turned to 90 degrees
- moved R3 253.5 mm to (347.3, -8.26), turned to -90 degrees
- moved C1 243.1 mm to (359.4, -24.8), turned to -90 degrees
- moved C6 239.0 mm to (364.4, -22.2), turned to -90 degrees
- moved C7 237.5 mm to (356.8, -24.8), turned to 90 degrees
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Routing:
- net +BATT: track 0.00 -> 1530.0 mm
- net +12V: track 34.6 -> 268.5 mm
- net Net-(Q21-Pad3): track 0.00 -> 95.6 mm
- net /Resistor Tree Large/12V Gate Driver14/GATE: track 0.00 -> 90.0 mm
- net /Resistor Tree Large/12V Gate Driver13/GATE: track 0.00 -> 89.5 mm
- net /Resistor Tree Large/12V Gate Driver12/GATE: track 0.00 -> 88.5 mm
- net Net-(Q36-Pad3): track 0.00 -> 83.4 mm
- net +5V: track 0.00 -> 73.9 mm
- net Net-(Q20-Pad3): track 0.00 -> 54.2 mm
- net +3V3: track 0.00 -> 53.2 mm
- net GND: track 29.2 -> 78.0 mm
- net Net-(Q35-Pad3): track 0.00 -> 45.9 mm
- net Net-(J5-PadA6): track 0.00 -> 41.3 mm
- net Net-(J5-PadA7): track 0.00 -> 40.9 mm
- net /Resistor Tree Large/12V Gate Driver11/GATE: track 0.00 -> 36.7 mm
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Other:
- board outline added: 189.9 x 289.6 mm

Commit message: fix: update pin assignment for transistors
Parts:
- moved J4 59.5 mm to (387.5, 233.0)
- moved J2 39.5 mm to (356.7, 233.0)
- moved R57 6.16 mm to (420.8, 141.6), turned to -90 degrees
- moved R60 4.00 mm to (415.7, 141.6), turned to -90 degrees
- moved J3 3.05 mm to (424.0, 233.0)
- turned R110 to 90 degrees
Connections:
- C1 pad 1: GND -> GNDA
- C10 pad 2: GND -> GNDA
- C11 pad 2: GND -> GNDA
- C12 pad 1: GND -> GNDA
- C13 pad 2: GND -> GNDA
- C2 pad 2: GND -> GNDA
- C3 pad 2: GND -> GNDA
- C4 pad 2: GND -> GNDA
- C5 pad 2: GND -> GNDA
- C6 pad 2: GND -> GNDA
- C7 pad 2: GND -> GNDA
- C8 pad 2: GND -> GNDA
- C9 pad 2: GND -> GNDA
- D1 pad 1: GND -> GNDA
- J1 pad 2: GND -> GNDA
- J2 pad 1: GND -> GNDA
- J4 pad 1: unconnected-(J4-Pad1) -> GND
- J5 pad A1B12: GND -> GNDA
- J5 pad B1A12: GND -> GNDA
- J5 pad S1: GND -> GNDA
- J5 pad S2: GND -> GNDA
- J5 pad S3: GND -> GNDA
- J5 pad S4: GND -> GNDA
- J6 pad 20: GND -> GNDA
- J7 pad 2: GND -> GNDA
- J8 pad 2: GND -> GNDA
- Q10 pad 2: GND -> Net-(Q10-Pad2)
- Q10 pad 3: Net-(Q10-Pad3) -> GND
- Q11 pad 2: GND -> Net-(Q11-Pad2)
- Q11 pad 3: Net-(Q11-Pad3) -> GND
- Q12 pad 2: GND -> Net-(Q12-Pad2)
- Q12 pad 3: Net-(Q12-Pad3) -> GND
- Q13 pad 2: GND -> Net-(Q13-Pad2)
- Q13 pad 3: Net-(Q13-Pad3) -> GND
- Q14 pad 2: GND -> Net-(Q14-Pad2)
- Q14 pad 3: Net-(Q14-Pad3) -> GND
- Q15 pad 2: GND -> Net-(Q15-Pad2)
- Q15 pad 3: Net-(Q15-Pad3) -> GND
- Q16 pad 2: GND -> Net-(Q16-Pad2)
- Q16 pad 3: Net-(Q16-Pad3) -> GND
- Q17 pad 2: GND -> Net-(Q17-Pad2)
- Q17 pad 3: Net-(Q17-Pad3) -> GND
- Q18 pad 2: GND -> Net-(Q18-Pad2)
- Q18 pad 3: Net-(Q18-Pad3) -> GND
- Q19 pad 2: GND -> Net-(Q19-Pad2)
- Q19 pad 3: Net-(Q19-Pad3) -> GND
- Q20 pad 2: GND -> Net-(Q20-Pad2)
- Q20 pad 3: Net-(Q20-Pad3) -> GND
- Q21 pad 2: GND -> Net-(Q21-Pad2)
- Q21 pad 3: Net-(Q21-Pad3) -> GND
- Q22 pad 2: GND -> Net-(Q22-Pad2)
- Q22 pad 3: Net-(Q22-Pad3) -> GND
- Q4 pad 2: GND -> Net-(Q4-Pad2)
- Q4 pad 3: Net-(Q4-Pad3) -> GND
- Q5 pad 2: GND -> Net-(Q5-Pad2)
- Q5 pad 3: Net-(Q5-Pad3) -> GND
- Q6 pad 2: GND -> Net-(Q6-Pad2)
- Q6 pad 3: Net-(Q6-Pad3) -> GND
- Q7 pad 2: GND -> Net-(Q7-Pad2)
- Q7 pad 3: Net-(Q7-Pad3) -> GND
- Q8 pad 2: GND -> Net-(Q8-Pad2)
- Q8 pad 3: Net-(Q8-Pad3) -> GND
- Q9 pad 2: GND -> Net-(Q9-Pad2)
- Q9 pad 3: Net-(Q9-Pad3) -> GND
- R10 pad 1: Net-(Q8-Pad3) -> Net-(Q8-Pad2)
- R11 pad 2: Net-(Q4-Pad3) -> Net-(Q4-Pad2)
- R12 pad 2: Net-(Q5-Pad3) -> Net-(Q5-Pad2)
- R13 pad 2: Net-(Q6-Pad3) -> Net-(Q6-Pad2)
- R14 pad 2: Net-(Q7-Pad3) -> Net-(Q7-Pad2)
- R15 pad 1: Net-(Q4-Pad3) -> Net-(Q4-Pad2)
- R16 pad 1: Net-(Q5-Pad3) -> Net-(Q5-Pad2)
- R17 pad 1: Net-(Q6-Pad3) -> Net-(Q6-Pad2)
- R18 pad 1: Net-(Q7-Pad3) -> Net-(Q7-Pad2)
- R19 pad 2: Net-(Q9-Pad3) -> Net-(Q9-Pad2)
- R2 pad 2: GND -> GNDA
- R20 pad 2: GND -> GNDA
- R23 pad 2: GND -> GNDA
- R26 pad 2: Net-(Q10-Pad3) -> Net-(Q10-Pad2)
- R27 pad 1: Net-(Q9-Pad3) -> Net-(Q9-Pad2)
- R28 pad 1: Net-(Q10-Pad3) -> Net-(Q10-Pad2)
- R29 pad 2: Net-(Q11-Pad3) -> Net-(Q11-Pad2)
- R30 pad 2: Net-(Q12-Pad3) -> Net-(Q12-Pad2)
- R31 pad 2: Net-(Q13-Pad3) -> Net-(Q13-Pad2)
- R32 pad 2: Net-(Q14-Pad3) -> Net-(Q14-Pad2)
- R33 pad 1: Net-(Q11-Pad3) -> Net-(Q11-Pad2)
- R34 pad 1: Net-(Q12-Pad3) -> Net-(Q12-Pad2)
- R35 pad 1: Net-(Q13-Pad3) -> Net-(Q13-Pad2)
- R36 pad 1: Net-(Q14-Pad3) -> Net-(Q14-Pad2)
- R37 pad 2: Net-(Q15-Pad3) -> Net-(Q15-Pad2)
- R38 pad 2: Net-(Q16-Pad3) -> Net-(Q16-Pad2)
- R39 pad 2: Net-(Q17-Pad3) -> Net-(Q17-Pad2)
- R4 pad 2: GND -> GNDA
- R40 pad 2: Net-(Q18-Pad3) -> Net-(Q18-Pad2)
- R41 pad 1: Net-(Q15-Pad3) -> Net-(Q15-Pad2)
- R42 pad 1: Net-(Q16-Pad3) -> Net-(Q16-Pad2)
- R43 pad 1: Net-(Q17-Pad3) -> Net-(Q17-Pad2)
- R44 pad 1: Net-(Q18-Pad3) -> Net-(Q18-Pad2)
- R45 pad 2: Net-(Q19-Pad3) -> Net-(Q19-Pad2)
- R46 pad 2: Net-(Q20-Pad3) -> Net-(Q20-Pad2)
- R47 pad 2: Net-(Q21-Pad3) -> Net-(Q21-Pad2)
- R48 pad 2: Net-(Q22-Pad3) -> Net-(Q22-Pad2)
- R49 pad 2: Net-(Q20-Pad3) -> Net-(Q20-Pad2)
- R50 pad 2: Net-(Q21-Pad3) -> Net-(Q21-Pad2)
- R51 pad 2: Net-(Q19-Pad3) -> Net-(Q19-Pad2)
- R52 pad 1: Net-(Q19-Pad3) -> Net-(Q19-Pad2)
- R53 pad 1: Net-(Q22-Pad3) -> Net-(Q22-Pad2)
- R54 pad 2: Net-(Q20-Pad3) -> Net-(Q20-Pad2)
- R55 pad 1: Net-(Q20-Pad3) -> Net-(Q20-Pad2)
- R56 pad 2: Net-(Q21-Pad3) -> Net-(Q21-Pad2)
- R57 pad 1: Net-(Q21-Pad3) -> Net-(Q21-Pad2)
- R58 pad 2: Net-(Q20-Pad3) -> Net-(Q20-Pad2)
- R59 pad 2: Net-(Q21-Pad3) -> Net-(Q21-Pad2)
- R60 pad 1: Net-(Q21-Pad3) -> Net-(Q21-Pad2)
- R61 pad 2: Net-(Q21-Pad3) -> Net-(Q21-Pad2)
- R62 pad 2: Net-(Q21-Pad3) -> Net-(Q21-Pad2)
- R63 pad 2: Net-(Q21-Pad3) -> Net-(Q21-Pad2)
- R64 pad 2: Net-(Q21-Pad3) -> Net-(Q21-Pad2)
- R9 pad 2: Net-(Q8-Pad3) -> Net-(Q8-Pad2)
- S1 pad 1: GND -> GNDA
- S2 pad 1: GND -> GNDA
- U1 pad 4: GND -> GNDA
- U1 pad 9: GND -> GNDA
- U2 pad 2: GND -> GNDA
- U3 pad 19: GND -> GNDA
- U3 pad 57: GND -> GNDA
- U4 pad 1: GND -> GNDA
- Y1 pad 2: GND -> GNDA
Routing:
- net +BATT: track 1530.0 -> 22.6 mm, vias 0 -> 1
- net Net-(Q21-Pad3): track 95.6 -> 0.00 mm
- net Net-(Q20-Pad3): track 54.2 -> 0.00 mm
- net Net-(Q20-Pad2): track 0.00 -> 46.5 mm
- net Net-(Q19-Pad3): track 34.2 -> 0.00 mm
- net Net-(Q19-Pad2): track 0.00 -> 26.6 mm
- net Net-(Q22-Pad3): track 23.9 -> 0.00 mm
- net Net-(Q8-Pad3): track 23.6 -> 0.00 mm
- net +12V: track 268.5 -> 291.0 mm
- net Net-(Q18-Pad3): track 20.9 -> 0.00 mm
- net Net-(Q14-Pad3): track 20.7 -> 0.00 mm
- net Net-(Q6-Pad3): track 20.7 -> 0.00 mm
- net Net-(Q10-Pad3): track 20.6 -> 0.00 mm
- net Net-(Q9-Pad3): track 20.4 -> 0.00 mm
- net Net-(Q15-Pad3): track 20.3 -> 0.00 mm
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- added copper zone on B.Cu, net +BATT
- added copper zone on F.Cu, net GND
- added copper zone on F.Cu, net Net-(Q21-Pad2)
Other:
- outline, holes or cut-outs redrawn

Commit message: Major rev 3
made edits
Parts:
- moved Q53 196.0 mm to (402.0, 211.8)
- moved R112 196.0 mm to (396.9, 211.8)
- moved R80 196.0 mm to (412.1, 211.8)
- moved D11 196.0 mm to (381.7, 214.3)
- moved Q37 196.0 mm to (407.1, 214.3)
- moved Q52 196.0 mm to (391.8, 214.3)
- moved Q54 196.0 mm to (402.0, 216.9)
- moved R111 196.0 mm to (396.9, 216.9)
- moved R113 196.0 mm to (386.7, 214.3)
- moved R79 196.0 mm to (427.0, 210.2)
- moved R84 196.0 mm to (423.0, 216.9)
- moved Q41 181.0 mm to (401.8, 181.6)
- moved Q51 181.0 mm to (401.8, 172.1)
- moved R100 181.0 mm to (396.8, 181.6)
- moved R108 181.0 mm to (396.8, 172.1)
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Routing:
- net GNDA: track 0.00 -> 567.5 mm, vias 0 -> 21
- net /Microcontroller/GPIO1: track 6.80 -> 360.9 mm, vias 0 -> 2
- net /Microcontroller/GPIO3: track 6.80 -> 340.5 mm, vias 0 -> 2
- net /Microcontroller/GPIO2: track 6.80 -> 332.1 mm, vias 0 -> 1
- net /Microcontroller/GPIO0: track 6.80 -> 300.1 mm
- net +12V: track 291.0 -> 581.3 mm, vias 0 -> 26
- net /Microcontroller/GPIO4: track 6.80 -> 281.0 mm, vias 0 -> 2
- net /Microcontroller/GPIO5: track 5.73 -> 207.9 mm, vias 0 -> 2
- net GND: track 84.8 -> 284.0 mm, vias 2 -> 29
- net /Microcontroller/GPIO6: track 5.73 -> 174.9 mm, vias 0 -> 3
- net /Microcontroller/GPIO7: track 5.73 -> 142.8 mm, vias 0 -> 2
- net /Microcontroller/GPIO12: track 11.7 -> 123.5 mm, vias 0 -> 2
- net /Microcontroller/GPIO8: track 5.73 -> 102.7 mm, vias 0 -> 2
- net /Microcontroller/GPIO9: track 5.73 -> 93.6 mm, vias 0 -> 2
- net /Microcontroller/GPIO10: track 5.73 -> 85.5 mm, vias 0 -> 2
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